File: PCBs/BuckLars/BuckPCB/BuckPCB.kicad_pcb (KiCad board)
At the start: 2 copper layers, 78.7 x 89.4 mm, 90 parts, among them Q1 IRLIZ44N, Q2 IRLIZ44N, Q3 IRLIZ44N, Q4 IRLIZ44N, U1 ESP32-WROOM-32D, U2 LT1936, U3 LF2304NTR, U4 LF2304NTR, U5 LT1936

Commit message: changed buck driver circuit
Parts:
- added D16: 1N4148WT, Diode_SMD:D_SOD-523, F.Cu at (162.0, 103.0)
- added D17: 1N4148WT, Diode_SMD:D_SOD-523, F.Cu at (162.4, 127.1)
- moved C9 1.16 mm to (159.2, 127.2)
Connections:
- U3 pad 3: Imeasure -> +5V
- U4 pad 3: Imeasure -> +5V
Routing:
- net +5V: track 121.6 -> 142.7 mm, vias 4 -> 6
- net Imeasure: track 106.9 -> 110.1 mm, vias 64 -> 66
- net Net-(D17-K): track 2.27 -> 4.64 mm
- net Net-(D16-K): track 2.43 -> 3.99 mm
- net GND: vias 298 -> 297
Other:
- board text added: "GND"
- board text added: "VIN"
- board text added: "VIN 7V-36V"
- board text added: "VOUT"
- board text removed: "+"
- board text removed: "-"
